Commit message: Added sensors plugins and modified intertial values

File: my_rb1_description/urdf/my_rb1_robot.urdf (robot description, URDF)
Before this commit: robot robot, 7 links, 6 joints
Links:
- removed link link_laser_scan
- added link front_laser, mass 0.5; collision cylinder length=0.0020 radius=0.005; visual cylinder length=0.0020 radius=0.005
Joints:
- joint joint_laser_scan_chassis: child link_laser_scan -> front_laser

Commit message: Modified URDF

File: my_rb1_description/urdf/my_rb1_robot.urdf (robot description, URDF)
Before this commit: robot robot, 7 links, 6 joints
Joints:
- joint joint_base_footprint: child base_footprint -> base_link; origin xyz=0.0 0.0 -0.15 rpy=0 0 0 -> xyz=0.0 0.0 0.15 rpy=0 0 0; parent base_link -> base_footprint
- joint joint_chassis_left_wheel: origin xyz=0 -0.2 -0.15 rpy=0 0 0 -> xyz=0 0.2 -0.15 rpy=0 0 0
- joint joint_chassis_right_wheel: origin xyz=0 0.2 -0.15 rpy=0 0 0 -> xyz=0 -0.2 -0.15 rpy=0 0 0

Commit message: Modified URDF and Implemented Rotate srv Node

File: my_rb1_description/urdf/my_rb1_robot.urdf (robot description, URDF)
Before this commit: robot robot, 7 links, 6 joints
Links:
- removed link link_back_caster_wheel
- removed link link_front_caster_wheel
- removed link link_left_wheel
- removed link link_right_wheel
- added link back_caster, mass 0.5; collision sphere radius=0.025; visual sphere radius=0.025
- added link front_caster, mass 0.5; collision sphere radius=0.025; visual sphere radius=0.025
- added link left_wheel, mass 1.5; collision cylinder length=0.03 radius=0.025; visual cylinder length=0.03 radius=0.025
- added link right_wheel, mass 1.5; collision cylinder length=0.03 radius=0.025; visual cylinder length=0.03 radius=0.025
- link base_link: mass 25 -> 20.5
- link front_laser: mass 0.5 -> None; geometry 
Joints:
- removed joint joint_base_footprint
- removed joint joint_chassis_back_caster_wheel
- removed joint joint_chassis_front_caster_wheel
- removed joint joint_chassis_left_wheel
- removed joint joint_chassis_right_wheel
- removed joint joint_laser_scan_chassis
- added joint base_link_back_caster_joint: type fixed, parent base_link, child back_caster, origin xyz=-0.1 0.0 -0.15 rpy=0 0 0
- added joint base_link_front_caster_joint: type fixed, parent base_link, child front_caster, origin xyz=0.1 0.0 -0.15 rpy=0 0 0
- added joint base_link_front_laser_joint: type fixed, parent base_link, child front_laser, origin xyz=0.25 0 0.075 rpy=3.14 0 0
- added joint base_link_left_wheel_joint: type continuous, parent base_link, child left_wheel, origin xyz=0 0.2 -0.15 rpy=0 0 0, axis 0 1 0
- added joint base_link_plate_joint: type fixed, parent base_footprint, child base_link, origin xyz=0 0 0.15 rpy=0 0 0
- added joint base_link_right_wheel_joint: type continuous, parent base_link, child right_wheel, origin xyz=0 -0.2 -0.15 rpy=0 0 0, axis 0 1 0
